Commit message: fix: update the URDF for the panda with FT

File: assets/industreal/urdf/industreal_franka.urdf (robot description, URDF)
Before this commit: robot panda, 12 links, 11 joints
Links:
- added link ft_sensor, mass 0.6; collision cylinder length=0.025 radius=0.042; visual cylinder length=0.025 radius=0.042
Joints:
- added joint ft_sensor_joint: type fixed, parent panda_link7, child ft_sensor, origin xyz=0 0 0.107 rpy=0 0 0
- joint panda_hand_joint: origin xyz=0 0 0.107 rpy=0 0 -0.7853981633974483 -> xyz=0 0 0.026 rpy=0 0 1.57079632679; parent panda_link7 -> ft_sensor

Commit message: fix: update the measured offsets

File: assets/industreal/urdf/industreal_franka.urdf (robot description, URDF)
Before this commit: robot panda, 13 links, 12 joints
Links:
- link ft_sensor: geometry collision cylinder length=0.068 radius=0.042; visual cylinder length=0.068 radius=0.042
Joints:
- joint panda_hand_joint: origin xyz=0 0 0.026 rpy=0 0 1.57079632679 -> xyz=0 0 0.068 rpy=0 0 1.57079632679
